File: Capteur_Graphite/Capteur_Graphite.kicad_sch (KiCad schematic)
At the start: 21 parts, among them J1 Power, J2 Digital/PWM, J3 Analog, J4 Digital/PWM, U1 LTC1050ACN8_PBF, U2 MCP41050

Commit message: Clear PCB
Parts:
- C3, C4: footprint Capacitor_THT:C_Rect_L7.5mm_W6.5mm_P5.00mm -> Capacitor_THT:C_Rect_L7.0mm_W4.5mm_P5.00mm
Changed lines of the file:
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@@
 			)
 		)
-		(property "Footprint" "Capacitor_THT:C_Rect_L7.5mm_W6.5mm_P5.00mm"
+		(property "Footprint" "Capacitor_THT:C_Rect_L7.0mm_W4.5mm_P5.00mm"
 			(at 135.5852 40.64 0)
 			(effects
@@
 			)
 		)
-		(property "Footprint" "Capacitor_THT:C_Rect_L7.5mm_W6.5mm_P5.00mm"
+		(property "Footprint" "Capacitor_THT:C_Rect_L7.0mm_W4.5mm_P5.00mm"
 			(at 172.4152 96.52 0)
 			(effects

Commit message: Schematique propre
Connections:
- net *10 is gone; now on net 10: J2.8 (Pin_8)
- net *11 is gone; now on net 11: J2.7 (Pin_7)
- net *5 is gone; now on net P5: J4.3 (Pin_3)
- net *9 is gone; now on net ServoOut: J2.9 (Pin_9)
- net +5V is gone; now on net +5: J1.5 (Pin_5)
- net 12 is gone; now on net 13: J2.6 (Pin_6)
- net 2 is gone; now on net P2: J4.6 (Pin_6)
- net 4 is gone; now on net P4: J4.4 (Pin_4)
- net SCL/A5 is gone; now on net SCL: J2.1 (Pin_1), J3.6 (Pin_6)
- net SDA/A4 is gone; now on net SDA: J2.2 (Pin_2), J3.5 (Pin_5)

Commit message: Fin de séance du 13 mars
Connections:
- net 13: no longer J2.6 (Pin_6)
- new net 12: J2.6 (Pin_6)
Changed lines of the file:
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@@
+	(wire
+		(pts
+			(xy 73.66 39.37) (xy 62.23 39.37)
+		)
+		(stroke
+			(width 0)
+			(type solid)
+		)
+	)
 	(wire
 		(pts
@@
 		(pts
 			(xy 34.29 59.69) (xy 21.59 59.69)
-		)
-		(stroke
-			(width 0)
-			(type solid)
-		)
-	)
-	(wire
-		(pts
-			(xy 62.23 39.37) (xy 74.93 39.37)
 		)
 		(stroke
@@
 	)
 	(label "12"
-		(at 74.93 39.37 180)
+		(at 73.66 39.37 180)
 		(fields_autoplaced yes)
 		(effects
@@
 	(global_label "13"
 		(shape bidirectional)
-		(at 74.93 39.37 0)
+		(at 73.66 36.83 0)
 		(fields_autoplaced yes)
 		(effects
@@
 		)
 		(property "Intersheetrefs" "${INTERSHEET_REFS}"
-			(at 81.4453 39.37 0)
+			(at 80.1753 36.83 0)
 			(effects
 				(font

Commit message: PCB fini
Connections:
- net +5: now also Bluetooth1.5 (VCC)
- net VCC: no longer Bluetooth1.5 (VCC)
Changed lines of the file:
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@@
 (kicad_sch
-	(version 20231120)
+	(version 20250114)
 	(generator "eeschema")
-	(generator_version "8.0")
+	(generator_version "9.0")
 	(paper "A4")
 	(title_block
 		(date "mar. 31 mars 2015")
 	)
+	(rectangle
+		(start 175.26 29.21)
+		(end 208.28 53.34)
+		(stroke
+			(width 0)
+			(type default)
+		)
+		(fill
+			(type none)
+		)
+	)
+	(rectangle
+		(start 121.92 17.78)
+		(end 167.64 55.88)
+		(stroke
+			(width 0)
+			(type default)
+		)
+		(fill
+			(type none)
+		)
+	)
+	(rectangle
+		(start 19.05 85.09)
+		(end 218.44 166.37)
+		(stroke
+			(width 0)
+			(type default)
+		)
+		(fill
+			(type none)
+		)
+	)
+	(rectangle
+		(start 80.01 16.51)
+		(end 111.76 40.64)
+		(stroke
+			(width 0)
+			(type default)
+		)
+		(fill
+			(type none)
+		)
+	)
+	(rectangle
+		(start 120.65 57.15)
+		(end 144.78 81.28)
+		(stroke
+			(width 0)
+			(type default)
+		)
+		(fill
+			(type none)
+		)
+	)
+	(rectangle
+		(start 77.47 46.99)
+		(end 118.11 81.28)
+		(stroke
+			(width 0)
+			(type default)
+		)
+		(fill
+			(type none)
+		)
+	)
+	(text "Amplificateur"
+		(exclude_from_sim no)
+		(at 25.908 128.016 0)
+		(effects
+			(font
+				(size 1.27 1.27)
+			)
+		)
+	)
+	(text "* Indicates a PWM-capable pin"
+		(exclude_from_sim no)
+		(at 177.8 180.34 0)
+		(effects
+			(font
+				(size 1.27 1.27)
+			)
+			(justify left bottom)
+		)
+	)
 	(junction
 		(at 134.62 33.02)
@@
 		)
 	)
-	(rectangle
-		(start 175.26 29.21)
-		(end 208.28 53.34)
-		(stroke
-			(width 0)
-			(type default)
-		)
-		(fill
-			(type none)
-		)
-	)
-	(rectangle
-		(start 121.92 17.78)
-		(end 167.64 55.88)
-		(stroke
-			(width 0)
-			(type default)
-		)
-		(fill
-			(type none)
-		)
-	)
-	(rectangle
-		(start 19.05 85.09)
-		(end 218.44 166.37)
-		(stroke
-			(width 0)
-			(type default)
-		)
-		(fill
-			(type none)
-		)
-	)
-	(rectangle
-		(start 80.01 16.51)
-		(end 111.76 40.64)
-		(stroke
-			(width 0)
-			(type default)
-		)
-		(fill
-			(type none)
-		)
-	)
-	(rectangle
-		(start 120.65 57.15)
-		(end 144.78 81.28)
-		(stroke
-			(width 0)
-			(type default)
-		)
-		(fill
-			(type none)
-		)
-	)
-	(rectangle
-		(start 77.47 46.99)
-		(end 118.11 81.28)
-		(stroke
-			(width 0)
-			(type default)
-		)
-		(fill
-			(type none)
-		)
-	)
-	(text "Amplificateur"
-		(exclude_from_sim no)
-		(at 25.908 128.016 0)
-		(effects
-			(font
-				(size 1.27 1.27)
-			)
-		)
-	)
-	(text "* Indicates a PWM-capable pin"
-		(exclude_from_sim no)
-		(at 177.8 180.34 0)
-		(effects
-			(font
-				(size 1.27 1.27)
-			)
-			(justify left bottom)
-		)
-	)
 	(label "RX{slash}0"
 		(at 74.93 77.47 180)
-		(fields_autoplaced yes)
 		(effects
 			(font
@@
 	(label "A2"
 		(at 21.59 64.77 0)
-		(fields_autoplaced yes)
 		(effects
 			(font
@@
 	(label "4"
 		(at 74.93 67.31 180)
-		(fields_autoplaced yes)
 		(effects
 			(font
@@
 	(label "2"
 		(at 74.93 72.39 180)
-		(fields_autoplaced yes)
 		(effects
 			(font
@@
 	(label "A3"
 		(at 21.59 67.31 0)
-		(fields_autoplaced yes)
 		(effects
 			(font
@@
 	(label "13"
 		(at 74.93 36.83 180)
-		(fields_autoplaced yes)
 		(effects
 			(font
@@
 	(label "12"
 		(at 73.66 39.37 180)
-		(fields_autoplaced yes)
 		(effects
 			(font
@@
 	(label "~{RESET}"
 		(at 19.05 36.83 0)
-		(fields_autoplaced yes)
 		(effects
 			(font
@@
 	(label "*10"
 		(at 74.93 44.45 180)
-		(fields_autoplaced yes)
 		(effects
 			(font
@@
 	(label "7"
 		(at 74.93 59.69 180)
-		(fields_autoplaced yes)
 		(effects
 			(font
@@
 	(label "SDA{slash}A4"
 		(at 74.93 29.21 180)
-		(fields_autoplaced yes)
 		(effects
 			(font
@@
 	(label "8"
 		(at 74.93 49.53 180)
-		(fields_autoplaced yes)
 		(effects
 			(font
@@
 	(label "*11"
 		(at 74.93 41.91 180)
-		(fields_autoplaced yes)
 		(effects
 			(font
@@
 	(label "*3"
 		(at 74.93 69.85 180)
-		(fields_autoplaced yes)
 		(effects
 			(font
@@
 	(label "A1"
 		(at 21.59 62.23 0)
-		(fields_autoplaced yes)
 		(effects
 			(font
@@
 	(label "TX{slash}1"
 		(at 74.93 74.93 180)
-		(fields_autoplaced yes)
 		(effects
 			(font
@@
 	(label "A0"
 		(at 21.59 59.69 0)
-		(fields_autoplaced yes)
 		(effects
 			(font
@@
 	(label "AREF"
 		(at 74.93 31.75 180)
-		(fields_autoplaced yes)
 		(effects
 			(font
@@
 	(label "Vin"
 		(at 26.67 26.67 270)
-		(fields_autoplaced yes)
 		(effects
 			(font
@@
 	(label "*6"
 		(at 74.93 62.23 180)
-		(fields_autoplaced yes)
 		(effects
 			(font
@@
 	(label "SCL{slash}A5"
 		(at 74.93 26.67 180)
-		(fields_autoplaced yes)
 		(effects
 			(font
@@
 	(label "*9"
 		(at 74.93 46.99 180)
-		(fields_autoplaced yes)
 		(effects
 			(font
@@
 	(label "*5"
 		(at 74.93 64.77 180)
-		(fields_autoplaced yes)
 		(effects
 			(font
@@
 	(label "IOREF"
 		(at 19.05 34.29 0)
-		(fields_autoplaced yes)
 		(effects
 			(font
@@
 	(label "SDA{slash}A4"
 		(at 21.59 69.85 0)
-		(fields_autoplaced yes)
 		(effects
 			(font
@@
 	(label "SCL{slash}A5"
 		(at 21.59 72.39 0)
-		(fields_autoplaced yes)
 		(effects
 			(font
@@
 		)
 	)
-	(global_label "VCC"
+	(global_label "+5"
 		(shape bidirectional)
 		(at 93.98 68.58 180)
@@
 		)
 		(property "Intersheetrefs" "${INTERSHEET_REFS}"
-			(at 86.2551 68.58 0)
+			(at 87.1018 68.58 0)
 			(effects
 				(font
@@
 		)
 	)
+	(embedded_fonts no)
 )

Commit message: Version Final du PCB + Gerber
Parts:
- Bluetooth1: footprint Ma_Lib_Empreinte_Projet_Capteur:HC05 -> Librairie empreinte:Bluetooth
- Capteur1: footprint Ma_Lib_Empreinte_Projet_Capteur:CapteurGraph -> Librairie empreinte:CapteurGraph
- Flex1: footprint Ma_Lib_Empreinte_Projet_Capteur:FlexSensor -> Librairie empreinte:FlexSensor
- OLED1: footprint Ma_Lib_Empreinte_Projet_Capteur:OLED -> Librairie empreinte:OLED
- Servor1: footprint Ma_Lib_Empreinte_Projet_Capteur:ServoMotor -> Librairie empreinte:ServoMotor
- U1, U2: footprint Ma_Lib_Empreinte_Projet_Capteur:LTC1050 -> Librairie empreinte:LTC1050
- U6: footprint Ma_Lib_Empreinte_Projet_Capteur:Rotatoire -> Librairie empreinte:Rotatoire
Changed lines of the file:
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@@
 			)
 		)
-		(property "Footprint" "Ma_Lib_Empreinte_Projet_Capteur:Rotatoire"
+		(property "Footprint" "Librairie empreinte:Rotatoire"
 			(at 148.59 36.83 0)
 			(effects
@@
 			)
 		)
-		(property "Footprint" "Ma_Lib_Empreinte_Projet_Capteur:OLED"
+		(property "Footprint" "Librairie empreinte:OLED"
 			(at 92.71 31.75 0)
 			(effects
@@
 			)
 		)
-		(property "Footprint" "Ma_Lib_Empreinte_Projet_Capteur:LTC1050"
+		(property "Footprint" "Librairie empreinte:LTC1050"
 			(at 101.6 99.06 0)
 			(effects
@@
 			)
 		)
-		(property "Footprint" "Ma_Lib_Empreinte_Projet_Capteur:CapteurGraph"
+		(property "Footprint" "Librairie empreinte:CapteurGraph"
 			(at 39.37 102.87 0)
 			(effects
@@
 			)
 		)
-		(property "Footprint" "Ma_Lib_Empreinte_Projet_Capteur:HC05"
+		(property "Footprint" "Librairie empreinte:Bluetooth"
 			(at 93.98 64.77 0)
 			(effects
@@
 			)
 		)
-		(property "Footprint" "Ma_Lib_Empreinte_Projet_Capteur:FlexSensor"
+		(property "Footprint" "Librairie empreinte:FlexSensor"
 			(at 134.62 68.58 0)
 			(effects
@@
 			)
 		)
-		(property "Footprint" "Ma_Lib_Empreinte_Projet_Capteur:ServoMotor"
+		(property "Footprint" "Librairie empreinte:ServoMotor"
 			(at 190.5 45.72 0)
 			(effects
@@
 			)
 		)
-		(property "Footprint" "Ma_Lib_Empreinte_Projet_Capteur:LTC1050"
+		(property "Footprint" "Librairie empreinte:LTC1050"
 			(at 55.88 139.7 0)
 			(effects

Commit message: Version Final corrigée du PCB
Parts:
- Rsensor1: footprint Resistor_THT:R_Axial_DIN0204_L3.6mm_D1.6mm_P1.90mm_Vertical -> Resistor_THT:R_Axial_DIN0309_L9.0mm_D3.2mm_P5.08mm_Vertical
Connections:
- net GND: now also Bluetooth1.1 (State), Bluetooth1.6 (Key), U1.1 (NC_2), U1.5 (EXTCLOCKINPUT), U1.8 (NC)
